Commit message: Refactor matrobot.xacro for improved structure

File: matrobot_description/urdf/matrobot.xacro (robot description, xacro)
@@ -1,4 +1,6 @@
 <?xml version="1.0" encoding="utf-8"?>
 <robot name="matrobot" xmlns:xacro="http://www.ros.org/wiki/xacro">
+  <xacro:property name="mesh_root" value="$(find matrobot_description)/meshes"/>
+  <!--mesh filename="file://${mesh_root}/base_link.STL" /--> <!--urdf oluşturduktan sonra visual kısma ekle-->
   <static>false</static>
   <!-- Properties -->
@@ -13,5 +15,5 @@
   <xacro:property name="caster_wheel_radius" value="${(wheel_radius - (base_height / 2)) / 2}" />
   <xacro:property name="caster_wheel_weight" value="0.5" />
-  <xacro:property name="wheel_separation" value="${base_width + wheel_length + 0.04}" />
+  <xacro:property name="wheel_separation" value="${base_width + wheel_length + 0.08}" />  <!--Gövde genişliği + (Teker genişliği/2)*2 + mil uzunluğu-->
   <xacro:property name="wheel_diameter" value="${wheel_radius}" />
   <xacro:property name="lidar_radius" value="0.0275"/>

Commit message: donanımsal sorun çözülmeye çalışıldı

File: matrobot_description/urdf/matrobot.xacro (robot description, xacro)
@@ -6,4 +6,5 @@
   <!-- Properties -->
   <xacro:include filename="$(find matrobot_description)/urdf/properties.xacro" />
+  <xacro:arg name="use_gazebo" default="false"/>
   <xacro:property name="base_width" value="0.34" />
   <xacro:property name="base_length" value="0.4" />
@@ -126,34 +127,4 @@
     <origin xyz="${(base_length / 2) - 0.05} 0 ${(base_height / 2) +0.05}" rpy="0 0 0"/>
   </joint>
-  <gazebo reference="lidar_link">
-    <sensor name="rplidar_s1" type="gpu_lidar">
-      <always_on>true</always_on>
-      <update_rate>10</update_rate>
-      <gz_frame_id>lidar_link</gz_frame_id>
-      <topic>/scan</topic>
-      <lidar>
-        <scan>
-          <horizontal>
-            <samples>640</samples>
-            <resolution>1</resolution>
-            <min_angle>-3.14159</min_angle>
-            <max_angle>3.14159</max_angle>
-          </horizontal>
-          <vertical>
-            <samples>1</samples>
-            <min_angle>0</min_angle>
-            <max_angle>0</max_angle>
-          </vertical>
-        </scan>
-        <range>
-          <min>0.15</min>
-          <max>40.0</max>
-          <resolution>0.01</resolution>
-        </range>
-      </lidar>
-      <!-- Ogre crash riskini azaltmak için -->
-      <visualize>false</visualize>
-    </sensor>
-  </gazebo>
   <!-- IMU Link & Joint -->
   <link name="imu_link"/>
@@ -164,93 +135,4 @@
     <axis xyz="0 1 0" />
   </joint>
-  <gazebo reference="imu_link">
-    <sensor name="imu_sensor" type="imu">
-      <always_on>1</always_on>
-      <update_rate>50</update_rate>
-      <topic>/imu</topic>
-      <gz_frame_id>imu_link</gz_frame_id>
-      <imu>
-        <enable_orientation>1</enable_orientation>
-        <angular_velocity>
-          <x>
-            <noise type="gaussian">
-              <mean>0</mean>
-              <stddev>0.009</stddev>
-              <bias_mean>0.00075</bias_mean>
-              <bias_stddev>0.005</bias_stddev>
-              <dynamic_bias_stddev>0.00002</dynamic_bias_stddev>
-              <dynamic_bias_correlation_time>400.0</dynamic_bias_correlation_time>
-              <precision>0.00025</precision>
-            </noise>
-          </x>
-          <y>
-            <noise type="gaussian">
-              <mean>0</mean>
-              <stddev>0.009</stddev>
-              <bias_mean>0.00075</bias_mean>
-              <bias_stddev>0.005</bias_stddev>
-              <dynamic_bias_stddev>0.00002</dynamic_bias_stddev>
-              <dynamic_bias_correlation_time>400.0</dynamic_bias_correlation_time>
-              <precision>0.00025</precision>
-            </noise>
-          </y>
-          <z>
-            <noise type="gaussian">
-              <mean>0</mean>
-              <stddev>0.009</stddev>
-              <bias_mean>0.00075</bias_mean>
-              <bias_stddev>0.005</bias_stddev>
-              <dynamic_bias_stddev>0.00002</dynamic_bias_stddev>
-              <dynamic_bias_correlation_time>400.0</dynamic_bias_correlation_time>
-              <precision>0.00025</precision>
-            </noise>
-          </z>
-        </angular_velocity>
-        <linear_acceleration>
-          <x>
-            <noise type="gaussian">
-              <mean>0</mean>
-              <stddev>0.021</stddev>
-              <bias_mean>0.05</bias_mean>
-              <bias_stddev>0.0075</bias_stddev>
-              <dynamic_bias_stddev>0.000375</dynamic_bias_stddev>
-              <dynamic_bias_correlation_time>175.0</dynamic_bias_correlation_time>
-              <precision>0.005</precision>
-            </noise>
-          </x>
-          <y>
-            <noise type="gaussian">
-              <mean>0</mean>
-              <stddev>0.021</stddev>
-              <bias_mean>0.05</bias_mean>
-              <bias_stddev>0.0075</bias_stddev>
-              <dynamic_bias_stddev>0.000375</dynamic_bias_stddev>
-              <dynamic_bias_correlation_time>175.0</dynamic_bias_correlation_time>
-              <precision>0.005</precision>
-            </noise>
-          </y>
-          <z>
-            <noise type="gaussian">
-              <mean>0</mean>
-              <stddev>0.021</stddev>
-              <bias_mean>0.05</bias_mean>
-              <bias_stddev>0.0075</bias_stddev>
-              <dynamic_bias_stddev>0.000375</dynamic_bias_stddev>
-              <dynamic_bias_correlation_time>175.0</dynamic_bias_correlation_time>
-              <precision>0.005</precision>
-            </noise>
-          </z>
-        </linear_acceleration>
-      </imu>
-    </sensor>
-  </gazebo>
-  <!-- Gazebo visual / friction settings -->
-  <xacro:macro name="gazebo_visual_settings" params="link_name color_name">
-    <gazebo reference="${link_name}">
-      <material>${color_name}</material>
-      <mu1>1.5</mu1>
-      <mu2>1.5</mu2>
-    </gazebo>
-  </xacro:macro>
   <!-- Instantiate all links -->
   <xacro:Wheel_Link name="left_wheel"  parent_link="base_link"
@@ -263,29 +145,150 @@
                       x="${(base_length / 2) - 0.02}" y="0.0"
                       z="-${((wheel_radius + (base_height / 2)) / 2 )}"/>
-  <xacro:gazebo_visual_settings link_name="base_link"       color_name="Gazebo/Black" />
-  <xacro:gazebo_visual_settings link_name="left_wheel_link"  color_name="Gazebo/Red" />
-  <xacro:gazebo_visual_settings link_name="right_wheel_link" color_name="Gazebo/Red" />
-  <!-- DiffDrive plugin -->
-  <gazebo>
-    <plugin filename="gz-sim-diff-drive-system"
-            name="gz::sim::systems::DiffDrive">
-      <update_rate>20</update_rate>
-      <left_joint>left_wheel_joint</left_joint>
-      <right_joint>right_wheel_joint</right_joint>
-      <wheel_separation>${wheel_separation}</wheel_separation>
-      <wheel_radius>${wheel_radius}</wheel_radius>
-      <topic>/cmd_vel</topic>
-      <odom_topic>/odometry/wheel</odom_topic>
-      <odom_publish_frequency>50</odom_publish_frequency>
-      <frame_id>odom</frame_id>
-      <child_frame_id>base_footprint</child_frame_id>
-    </plugin>
-  </gazebo>
-  <!-- JointStatePublisher plugin -->
-  <gazebo>
-    <plugin filename="gz-sim-joint-state-publisher-system"
-            name="gz::sim::systems::JointStatePublisher">
-      <topic>/joint_states</topic>
-    </plugin>
-  </gazebo>
+	<!-- Gazebo visual / friction settings -->
+	<xacro:macro name="gazebo_visual_settings" params="link_name color_name">
+	  <gazebo reference="${link_name}">
+	    <material>${color_name}</material>
+	    <mu1>1.5</mu1>
+	    <mu2>1.5</mu2>
+	  </gazebo>
+	</xacro:macro>
+	<xacro:if value="$(arg use_gazebo)">
+		<gazebo reference="lidar_link">
+		  <sensor name="rplidar_s1" type="gpu_lidar">
+		    <always_on>true</always_on>
+		    <update_rate>10</update_rate>
+		    <gz_frame_id>lidar_link</gz_frame_id>
+		    <topic>/scan</topic>
+		    <lidar>
+		      <scan>
+		        <horizontal>
+		          <samples>640</samples>
+		          <resolution>1</resolution>
+		          <min_angle>-3.14159</min_angle>
+		          <max_angle>3.14159</max_angle>
+		        </horizontal>
+		        <vertical>
+		          <samples>1</samples>
+		          <min_angle>0</min_angle>
+		          <max_angle>0</max_angle>
+		        </vertical>
+		      </scan>
+		      <range>
+		        <min>0.15</min>
+		        <max>40.0</max>
+		        <resolution>0.01</resolution>
+		      </range>
+		    </lidar>
+		    <!-- Ogre crash riskini azaltmak için -->
+		    <visualize>false</visualize>
+		  </sensor>
+		</gazebo>
+		<gazebo reference="imu_link">
+		  <sensor name="imu_sensor" type="imu">
+		    <always_on>1</always_on>
+		    <update_rate>50</update_rate>
+		    <topic>/imu</topic>
+		    <gz_frame_id>imu_link</gz_frame_id>
+		    <imu>
+		      <enable_orientation>1</enable_orientation>
+		      <angular_velocity>
+		        <x>
+		          <noise type="gaussian">
+		            <mean>0</mean>
+		            <stddev>0.009</stddev>
+		            <bias_mean>0.00075</bias_mean>
+		            <bias_stddev>0.005</bias_stddev>
+		            <dynamic_bias_stddev>0.00002</dynamic_bias_stddev>
+		            <dynamic_bias_correlation_time>400.0</dynamic_bias_correlation_time>
+		            <precision>0.00025</precision>
+		          </noise>
+		        </x>
+		        <y>
+		          <noise type="gaussian">
+		            <mean>0</mean>
+		            <stddev>0.009</stddev>
+		            <bias_mean>0.00075</bias_mean>
+		            <bias_stddev>0.005</bias_stddev>
+		            <dynamic_bias_stddev>0.00002</dynamic_bias_stddev>
+		            <dynamic_bias_correlation_time>400.0</dynamic_bias_correlation_time>
+		            <precision>0.00025</precision>
+		          </noise>
+		        </y>
+		        <z>
+		          <noise type="gaussian">
+		            <mean>0</mean>
+		            <stddev>0.009</stddev>
+		            <bias_mean>0.00075</bias_mean>
+		            <bias_stddev>0.005</bias_stddev>
+		            <dynamic_bias_stddev>0.00002</dynamic_bias_stddev>
+		            <dynamic_bias_correlation_time>400.0</dynamic_bias_correlation_time>
+		            <precision>0.00025</precision>
+		          </noise>
+		        </z>
+		      </angular_velocity>
+		      <linear_acceleration>
+		        <x>
+		          <noise type="gaussian">
+		            <mean>0</mean>
+		            <stddev>0.021</stddev>
+		            <bias_mean>0.05</bias_mean>
+		            <bias_stddev>0.0075</bias_stddev>
+		            <dynamic_bias_stddev>0.000375</dynamic_bias_stddev>
+		            <dynamic_bias_correlation_time>175.0</dynamic_bias_correlation_time>
+		            <precision>0.005</precision>
+		          </noise>
+		        </x>
+		        <y>
+		          <noise type="gaussian">
+		            <mean>0</mean>
+		            <stddev>0.021</stddev>
+		            <bias_mean>0.05</bias_mean>
+		            <bias_stddev>0.0075</bias_stddev>
+		            <dynamic_bias_stddev>0.000375</dynamic_bias_stddev>
+		            <dynamic_bias_correlation_time>175.0</dynamic_bias_correlation_time>
+		            <precision>0.005</precision>
+		          </noise>
+		        </y>
+		        <z>
+		          <noise type="gaussian">
+		            <mean>0</mean>
+		            <stddev>0.021</stddev>
+		            <bias_mean>0.05</bias_mean>
+		            <bias_stddev>0.0075</bias_stddev>
+		            <dynamic_bias_stddev>0.000375</dynamic_bias_stddev>
+		            <dynamic_bias_correlation_time>175.0</dynamic_bias_correlation_time>
+		            <precision>0.005</precision>
+		          </noise>
+		        </z>
+		      </linear_acceleration>
+		    </imu>
+		  </sensor>
+		</gazebo>
+		<!-- DiffDrive plugin -->
+		<gazebo>
+		  <plugin filename="gz-sim-diff-drive-system"
+		          name="gz::sim::systems::DiffDrive">
+		    <update_rate>20</update_rate>
+		    <left_joint>left_wheel_joint</left_joint>
+		    <right_joint>right_wheel_joint</right_joint>
+		    <wheel_separation>${wheel_separation}</wheel_separation>
+		    <wheel_radius>${wheel_radius}</wheel_radius>
+		    <topic>/cmd_vel</topic>
+		    <odom_topic>/odometry/wheel</odom_topic>
+		    <odom_publish_frequency>50</odom_publish_frequency>
+		    <frame_id>odom</frame_id>
+		    <child_frame_id>base_footprint</child_frame_id>
+		  </plugin>
+		</gazebo>
+		<!-- JointStatePublisher plugin -->
+		<gazebo>
+		  <plugin filename="gz-sim-joint-state-publisher-system"
+		          name="gz::sim::systems::JointStatePublisher">
+		    <topic>/joint_states</topic>
+		  </plugin>
+		</gazebo>
+		<xacro:gazebo_visual_settings link_name="base_link"       color_name="Gazebo/Black" />
+		<xacro:gazebo_visual_settings link_name="left_wheel_link"  color_name="Gazebo/Red" />
+		<xacro:gazebo_visual_settings link_name="right_wheel_link" color_name="Gazebo/Red" />
+	</xacro:if>
 </robot>

Commit message: donanım sorunu çözüldü. otomotik olarak kumandaya bağlanma ve kumanda ile kontrol eklenildi. nav2 params düzenlenildi

File: matrobot_description/urdf/matrobot.xacro (robot description, xacro)
@@ -111,15 +111,5 @@
   </xacro:macro>
   <!-- LIDAR Link & Joint -->
-  <link name="lidar_link">
-    <visual>
-      <origin xyz="0 0 0" rpy="0 0 0"/>
-      <geometry>
-        <mesh filename="file://$(find matrobot_description)/meshes/LIDAR.STL"/>
-      </geometry>
-      <material name="Gray">
-        <color rgba="0.75 0.75 0.75 1"/>
-      </material>
-    </visual>
-  </link>
+  <link name="lidar_link"/>
   <joint name="lidar_joint" type="fixed">
     <parent link="base_link"/>

Commit message: Update RViz configuration and adjust URDF properties for wheel dimensions and EKF parameters

File: matrobot_description/urdf/matrobot.xacro (robot description, xacro)
@@ -17,5 +17,5 @@
   <xacro:property name="caster_wheel_weight" value="0.5" />
   <xacro:property name="wheel_separation" value="${base_width + wheel_length + 0.08}" />  <!--Gövde genişliği + (Teker genişliği/2)*2 + mil uzunluğu-->
-  <xacro:property name="wheel_diameter" value="${wheel_radius}" />
+  <xacro:property name="wheel_diameter" value="${wheel_radius*2}" />
   <xacro:property name="lidar_radius" value="0.0275"/>
   <xacro:property name="lidar_height" value="0.04"/>
@@ -197,5 +197,5 @@
 		    <right_joint>right_wheel_joint</right_joint>
 		    <wheel_separation>${wheel_separation}</wheel_separation>
-		    <wheel_radius>${wheel_radius*2}</wheel_radius>
+		    <wheel_radius>${wheel_radius}</wheel_radius>
 		    <topic>/cmd_vel</topic>
 		    <odom_topic>/odometry/wheel</odom_topic>
